Commit message: arrange_axis

File: urdf/meta_arm.xacro (robot description, xacro)
@@ -6,7 +6,7 @@
 <link name="base_link">
   <inertial>
-    <origin xyz="-0.025593295674179693 -1.4061506970768674e-07 -0.010575799541855295" rpy="0 0 0"/>
+    <origin xyz="0.04958603260545487 0.3095418958770004 -0.33079876003291586" rpy="0 0 0"/>
     <mass value="0.06897369054613131"/>
-    <inertia ixx="4e-05" iyy="2.4e-05" izz="3.7e-05" ixy="0.0" iyz="0.0" ixz="-0.0"/>
+    <inertia ixx="4e-05" iyy="3.7e-05" izz="2.4e-05" ixy="0.0" iyz="0.0" ixz="-0.0"/>
   </inertial>
   <visual>
@@ -26,12 +26,132 @@
 <link name="link1_1">
   <inertial>
-    <origin xyz="0.023823701874984372 0.00027593219494978304 -0.02007724695428276" rpy="0 0 0"/>
+    <origin xyz="-0.023823964943709013 -0.020077551535427063 0.00027631277710354896" rpy="0 0 0"/>
     <mass value="0.09271114035136588"/>
-    <inertia ixx="5.9e-05" iyy="5.8e-05" izz="4.1e-05" ixy="-0.0" iyz="1e-06" ixz="0.0"/>
+    <inertia ixx="5.9e-05" iyy="4.1e-05" izz="5.8e-05" ixy="-0.0" iyz="1e-06" ixz="0.0"/>
+  </inertial>
+  <visual>
+    <origin xyz="-0.023993 -0.320118 0.330799" rpy="0 0 0"/>
+    <geometry>
+      <mesh filename="package://meta_arm_description/meshes/link1_1.stl" scale="0.001 0.001 0.001"/>
+    </geometry>
+    <material name="silver"/>
+  </visual>
+  <collision>
+    <origin xyz="-0.023993 -0.320118 0.330799" rpy="0 0 0"/>
+    <geometry>
+      <mesh filename="package://meta_arm_description/meshes/link1_1.stl" scale="0.001 0.001 0.001"/>
+    </geometry>
+  </collision>
+</link>
+<link name="link2_1">
+  <inertial>
+    <origin xyz="0.001185208127494953 -0.07376276671765236 -0.02120866884265743" rpy="0 0 0"/>
+    <mass value="0.1471165562988085"/>
+    <inertia ixx="0.000156" iyy="0.000101" izz="0.000149" ixy="2e-06" iyz="-0.0" ixz="0.0"/>
+  </inertial>
+  <visual>
+    <origin xyz="7e-06 -0.271618 0.308799" rpy="0 0 0"/>
+    <geometry>
+      <mesh filename="package://meta_arm_description/meshes/link2_1.stl" scale="0.001 0.001 0.001"/>
+    </geometry>
+    <material name="silver"/>
+  </visual>
+  <collision>
+    <origin xyz="7e-06 -0.271618 0.308799" rpy="0 0 0"/>
+    <geometry>
+      <mesh filename="package://meta_arm_description/meshes/link2_1.stl" scale="0.001 0.001 0.001"/>
+    </geometry>
+  </collision>
+</link>
+<link name="link3_1">
+  <inertial>
+    <origin xyz="-0.00041770484096615454 -0.10687879907009373 -0.0014259845445979136" rpy="0 0 0"/>
+    <mass value="0.10507743775617534"/>
+    <inertia ixx="0.000374" iyy="6.7e-05" izz="0.000374" ixy="-2e-06" iyz="-6e-06" ixz="0.0"/>
+  </inertial>
+  <visual>
+    <origin xyz="7e-06 -0.165618 0.329999" rpy="0 0 0"/>
+    <geometry>
+      <mesh filename="package://meta_arm_description/meshes/link3_1.stl" scale="0.001 0.001 0.001"/>
+    </geometry>
+    <material name="silver"/>
+  </visual>
+  <collision>
+    <origin xyz="7e-06 -0.165618 0.329999" rpy="0 0 0"/>
+    <geometry>
+      <mesh filename="package://meta_arm_description/meshes/link3_1.stl" scale="0.001 0.001 0.001"/>
+    </geometry>
+  </collision>
+</link>
+<link name="link4_1">
+  <inertial>
+    <origin xyz="0.020990707423285012 -0.0011925827569629456 0.07420496497953893" rpy="0 0 0"/>
+    <mass value="0.14623926771463272"/>
+    <inertia ixx="0.000144" iyy="0.000151" izz="0.0001" ixy="-0.0" iyz="2e-06" ixz="0.0"/>
+  </inertial>
+  <visual>
+    <origin xyz="0.021007 -0.0 0.33" rpy="0 0 0"/>
+    <geometry>
+      <mesh filename="package://meta_arm_description/meshes/link4_1.stl" scale="0.001 0.001 0.001"/>
+    </geometry>
+    <material name="silver"/>
+  </visual>
+  <collision>
+    <origin xyz="0.021007 -0.0 0.33" rpy="0 0 0"/>
+    <geometry>
+      <mesh filename="package://meta_arm_description/meshes/link4_1.stl" scale="0.001 0.001 0.001"/>
+    </geometry>
+  </collision>
+</link>
+<link name="link5_1">
+  <inertial>
+    <origin xyz="0.0004923916310237038 -1.4584999847711042e-05 0.11974132035335527" rpy="0 0 0"/>
+    <mass value="0.09246059265961544"/>
+    <inertia ixx="0.000458" iyy="0.00046" izz="5.8e-05" ixy="0.0" iyz="0.0" ixz="-3e-06"/>
+  </inertial>
+  <visual>
+    <origin xyz="7e-06 -0.0 0.224" rpy="0 0 0"/>
+    <geometry>
+      <mesh filename="package://meta_arm_description/meshes/link5_1.stl" scale="0.001 0.001 0.001"/>
+    </geometry>
+    <material name="silver"/>
+  </visual>
+  <collision>
+    <origin xyz="7e-06 -0.0 0.224" rpy="0 0 0"/>
+    <geometry>
+      <mesh filename="package://meta_arm_description/meshes/link5_1.stl" scale="0.001 0.001 0.001"/>
+    </geometry>
+  </collision>
+</link>
+<link name="link6_1">
+  <inertial>
+    <origin xyz="-0.02100001951500266 -8.579875966970071e-10 0.018539639017980714" rpy="0 0 0"/>
+    <mass value="0.029206480233661163"/>
+    <inertia ixx="1.1e-05" iyy="2.4e-05" izz="2.3e-05" ixy="-0.0" iyz="-0.0" ixz="0.0"/>
+  </inertial>
+  <visual>
+    <origin xyz="-0.021 -0.0 0.035" rpy="0 0 0"/>
+    <geometry>
+      <mesh filename="package://meta_arm_description/meshes/link6_1.stl" scale="0.001 0.001 0.001"/>
+    </geometry>
+    <material name="silver"/>
+  </visual>
+  <collision>
+    <origin xyz="-0.021 -0.0 0.035" rpy="0 0 0"/>
+    <geometry>
+      <mesh filename="package://meta_arm_description/meshes/link6_1.stl" scale="0.001 0.001 0.001"/>
+    </geometry>
+  </collision>
+</link>
+<link name="point_2">
+  <inertial>
+    <origin xyz="5.867230312706084e-14 1.489363048445824e-07 0.0012867771027078323" rpy="0 0 0"/>
+    <mass value="0.0006569528428977285"/>
+    <inertia ixx="0.0" iyy="0.0" izz="0.0" ixy="0.0" iyz="-0.0" ixz="-0.0"/>
   </inertial>
   <visual>
     <origin xyz="-0.0 0.0 0.0" rpy="0 0 0"/>
     <geometry>
-      <mesh filename="package://meta_arm_description/meshes/link1_1.stl" scale="0.001 0.001 0.001"/>
+      <mesh filename="package://meta_arm_description/meshes/point_2.stl" scale="0.001 0.001 0.001"/>
     </geometry>
     <material name="silver"/>
@@ -40,175 +160,55 @@
     <origin xyz="-0.0 0.0 0.0" rpy="0 0 0"/>
     <geometry>
-      <mesh filename="package://meta_arm_description/meshes/link1_1.stl" scale="0.001 0.001 0.001"/>
-    </geometry>
-  </collision>
-</link>
-<link name="link2_1">
-  <inertial>
-    <origin xyz="-0.0011854711962196625 -0.02120904942481134 -0.0737624621365079" rpy="0 0 0"/>
-    <mass value="0.1471165562988085"/>
-    <inertia ixx="0.000156" iyy="0.000149" izz="0.000101" ixy="-0.0" iyz="-0.0" ixz="-2e-06"/>
-  </inertial>
-  <visual>
-    <origin xyz="-0.024 -0.022 0.0485" rpy="0 0 0"/>
-    <geometry>
-      <mesh filename="package://meta_arm_description/meshes/link2_1.stl" scale="0.001 0.001 0.001"/>
-    </geometry>
-    <material name="silver"/>
-  </visual>
-  <collision>
-    <origin xyz="-0.024 -0.022 0.0485" rpy="0 0 0"/>
-    <geometry>
-      <mesh filename="package://meta_arm_description/meshes/link2_1.stl" scale="0.001 0.001 0.001"/>
-    </geometry>
-  </collision>
-</link>
-<link name="link3_1">
-  <inertial>
-    <origin xyz="0.00041744177224129625 -0.0014263651267520114 -0.10687849448894896" rpy="0 0 0"/>
-    <mass value="0.10507743775617534"/>
-    <inertia ixx="0.000374" iyy="0.000374" izz="6.7e-05" ixy="-0.0" iyz="-6e-06" ixz="2e-06"/>
-  </inertial>
-  <visual>
-    <origin xyz="-0.024 -0.0008 0.1545" rpy="0 0 0"/>
-    <geometry>
-      <mesh filename="package://meta_arm_description/meshes/link3_1.stl" scale="0.001 0.001 0.001"/>
-    </geometry>
-    <material name="silver"/>
-  </visual>
-  <collision>
-    <origin xyz="-0.024 -0.0008 0.1545" rpy="0 0 0"/>
-    <geometry>
-      <mesh filename="package://meta_arm_description/meshes/link3_1.stl" scale="0.001 0.001 0.001"/>
-    </geometry>
-  </collision>
-</link>
-<link name="link4_1">
-  <inertial>
-    <origin xyz="-0.02099097049201124 -0.001192963339153154 -0.07420466039839108" rpy="0 0 0"/>
-    <mass value="0.14623926771463272"/>
-    <inertia ixx="0.000144" iyy="0.000151" izz="0.0001" ixy="0.0" iyz="-2e-06" ixz="0.0"/>
-  </inertial>
-  <visual>
-    <origin xyz="-0.045 -0.000799 0.320118" rpy="0 0 0"/>
-    <geometry>
-      <mesh filename="package://meta_arm_description/meshes/link4_1.stl" scale="0.001 0.001 0.001"/>
-    </geometry>
-    <material name="silver"/>
-  </visual>
-  <collision>
-    <origin xyz="-0.045 -0.000799 0.320118" rpy="0 0 0"/>
-    <geometry>
-      <mesh filename="package://meta_arm_description/meshes/link4_1.stl" scale="0.001 0.001 0.001"/>
-    </geometry>
-  </collision>
-</link>
-<link name="link5_1">
-  <inertial>
-    <origin xyz="-0.0004926546997525288 -1.4965582042404321e-05 -0.1197410157722072" rpy="0 0 0"/>
-    <mass value="0.09246059265961544"/>
-    <inertia ixx="0.000458" iyy="0.00046" izz="5.8e-05" ixy="-0.0" iyz="-0.0" ixz="-3e-06"/>
-  </inertial>
-  <visual>
-    <origin xyz="-0.024 -0.000799 0.426118" rpy="0 0 0"/>
-    <geometry>
-      <mesh filename="package://meta_arm_description/meshes/link5_1.stl" scale="0.001 0.001 0.001"/>
-    </geometry>
-    <material name="silver"/>
-  </visual>
-  <collision>
-    <origin xyz="-0.024 -0.000799 0.426118" rpy="0 0 0"/>
-    <geometry>
-      <mesh filename="package://meta_arm_description/meshes/link5_1.stl" scale="0.001 0.001 0.001"/>
-    </geometry>
-  </collision>
-</link>
-<link name="link6_1">
-  <inertial>
-    <origin xyz="0.020999756446272243 -3.81440184788937e-07 -0.01853933443683209" rpy="0 0 0"/>
-    <mass value="0.029206480233661163"/>
-    <inertia ixx="1.1e-05" iyy="2.4e-05" izz="2.3e-05" ixy="0.0" iyz="0.0" ixz="0.0"/>
-  </inertial>
-  <visual>
-    <origin xyz="-0.002993 -0.000799 0.615118" rpy="0 0 0"/>
-    <geometry>
-      <mesh filename="package://meta_arm_description/meshes/link6_1.stl" scale="0.001 0.001 0.001"/>
-    </geometry>
-    <material name="silver"/>
-  </visual>
-  <collision>
-    <origin xyz="-0.002993 -0.000799 0.615118" rpy="0 0 0"/>
-    <geometry>
-      <mesh filename="package://meta_arm_description/meshes/link6_1.stl" scale="0.001 0.001 0.001"/>
-    </geometry>
-  </collision>
-</link>
-<link name="point_2">
-  <inertial>
-    <origin xyz="-2.630687893113992e-07 -2.3164589293999446e-07 -0.0012864725215591122" rpy="0 0 0"/>
-    <mass value="0.0006569528428977285"/>
-    <inertia ixx="0.0" iyy="0.0" izz="0.0" ixy="-0.0" iyz="0.0" ixz="-0.0"/>
-  </inertial>
-  <visual>
-    <origin xyz="-0.023993 -0.000799 0.650118" rpy="0 0 0"/>
-    <geometry>
       <mesh filename="package://meta_arm_description/meshes/point_2.stl" scale="0.001 0.001 0.001"/>
     </geometry>
-    <material name="silver"/>
-  </visual>
-  <collision>
-    <origin xyz="-0.023993 -0.000799 0.650118" rpy="0 0 0"/>
-    <geometry>
-      <mesh filename="package://meta_arm_description/meshes/point_2.stl" scale="0.001 0.001 0.001"/>
-    </geometry>
   </collision>
 </link>
 <joint name="joint1" type="revolute">
-  <origin xyz="0.0 0.0 0.0" rpy="0 0 0"/>
+  <origin xyz="0.023993 0.320118 -0.330799" rpy="0 0 0"/>
   <parent link="base_link"/>
   <child link="link1_1"/>
-  <axis xyz="1.0 -0.0 -0.0"/>
+  <axis xyz="-1.0 0.0 0.0"/>
   <limit upper="1.570796" lower="-1.570796" effort="100" velocity="100"/>
 </joint>
 <joint name="joint2" type="revolute">
-  <origin xyz="0.024 0.022 -0.0485" rpy="0 0 0"/>
+  <origin xyz="-0.024 -0.0485 0.022" rpy="0 0 0"/>
   <parent link="link1_1"/>
   <child link="link2_1"/>
-  <axis xyz="-0.0 1.0 0.0"/>
+  <axis xyz="0.0 0.0 1.0"/>
   <limit upper="0.0" lower="-1.570796" effort="100" velocity="100"/>
 </joint>
 <joint name="joint3" type="revolute">
-  <origin xyz="0.0 -0.0212 -0.106" rpy="0 0 0"/>
+  <origin xyz="0.0 -0.106 -0.0212" rpy="0 0 0"/>
   <parent link="link2_1"/>
   <child link="link3_1"/>
-  <axis xyz="-0.0 -0.0 -1.0"/>
+  <axis xyz="0.0 -1.0 0.0"/>
   <limit upper="0.0" lower="-1.745329" effort="100" velocity="100"/>
 </joint>
 <joint name="joint4" type="revolute">
-  <origin xyz="0.021 -1e-06 -0.165618" rpy="0 0 0"/>
+  <origin xyz="-0.021 -0.165618 -1e-06" rpy="0 0 0"/>
   <parent link="link3_1"/>
   <child link="link4_1"/>
-  <axis xyz="1.0 -0.0 -0.0"/>
+  <axis xyz="-1.0 -0.0 -0.0"/>
   <limit upper="1.745329" lower="0.0" effort="100" velocity="100"/>
 </joint>
 <joint name="joint5" type="revolute">
-  <origin xyz="-0.021 0.0 -0.106" rpy="0 0 0"/>
+  <origin xyz="0.021 0.0 0.106" rpy="0 0 0"/>
   <parent link="link4_1"/>
   <child link="link5_1"/>
-  <axis xyz="-0.0 -0.0 -1.0"/>
+  <axis xyz="0.0 0.0 1.0"/>
   <limit upper="0.0" lower="-3.141593" effort="100" velocity="100"/>
 </joint>
 <joint name="joint6" type="revolute">
-  <origin xyz="-0.021007 0.0 -0.189" rpy="0 0 0"/>
+  <origin xyz="0.021007 0.0 0.189" rpy="0 0 0"/>
   <parent link="link5_1"/>
   <child link="link6_1"/>
-  <axis xyz="-1.0 -0.0 0.0"/>
+  <axis xyz="1.0 -0.0 0.0"/>
   <limit upper="1.570796" lower="-1.570796" effort="100" velocity="100"/>
 </joint>
 <joint name="point" type="revolute">
-  <origin xyz="0.021 0.0 -0.035" rpy="0 0 0"/>
+  <origin xyz="-0.021 -0.0 0.035" rpy="0 0 0"/>
   <parent link="link6_1"/>
   <child link="point_2"/>
-  <axis xyz="-0.0 -0.0 -1.0"/>
+  <axis xyz="0.0 -0.0 1.0"/>
   <limit upper="0.00001" lower="0.0" effort="100" velocity="100"/>
 </joint>

Commit message: invere_done??

File: urdf/meta_arm.xacro (robot description, xacro)
@@ -183,5 +183,5 @@
   <child link="link3_1"/>
   <axis xyz="0.0 -1.0 0.0"/>
-  <limit upper="0.0" lower="-1.745329" effort="100" velocity="100"/>
+  <limit upper="2.617994" lower="-2.617994" effort="100" velocity="100"/>
 </joint>
 <joint name="joint4" type="revolute">
@@ -190,5 +190,5 @@
   <child link="link4_1"/>
   <axis xyz="-1.0 -0.0 -0.0"/>
-  <limit upper="1.745329" lower="0.0" effort="100" velocity="100"/>
+  <limit upper="0.0" lower="-1.745329" effort="100" velocity="100"/>
 </joint>
 <joint name="joint5" type="revolute">
@@ -197,5 +197,5 @@
   <child link="link5_1"/>
   <axis xyz="0.0 0.0 1.0"/>
-  <limit upper="0.0" lower="-3.141593" effort="100" velocity="100"/>
+  <limit upper="2.617994" lower="-2.617994" effort="100" velocity="100"/>
 </joint>
 <joint name="joint6" type="revolute">
@@ -206,5 +206,5 @@
   <limit upper="1.570796" lower="-1.570796" effort="100" velocity="100"/>
 </joint>
-<joint name="point" type="revolute">
+<joint name="point" type="fixed">
   <origin xyz="-0.021 -0.0 0.035" rpy="0 0 0"/>
   <parent link="link6_1"/>
