Commit message: r_l_arm_testing

File: urdf/Meta_arm_L.xacro (robot description, xacro)
@@ -190,5 +190,5 @@
   <child link="link4_1"/>
   <axis xyz="2.2e-05 0.999994 -0.003491"/>
-  <limit upper="0.0" lower="-2.181662" effort="100" velocity="100"/>
+  <limit upper="1.745329" lower="-0.872665" effort="100" velocity="100"/>
 </joint>
 <joint name="joint5" type="revolute">
@@ -206,5 +206,5 @@
   <limit upper="1.570796" lower="-1.570796" effort="100" velocity="100"/>
 </joint>
-<joint name="point" type="revolute">
+<joint name="point" type="fixed">
   <origin xyz="0.035 0.021 0.000142" rpy="0 0 0"/>
   <parent link="link6_1"/>

File: urdf/Meta_arm_R.xacro (robot description, xacro)
@@ -190,5 +190,5 @@
   <child link="link4_1"/>
   <axis xyz="0.001482 -0.99999 0.004202"/>
-  <limit upper="2.181662" lower="0.0" effort="100" velocity="100"/>
+  <limit upper="0.872665" lower="-1.745329" effort="100" velocity="100"/>
 </joint>
 <joint name="joint5" type="revolute">
@@ -206,5 +206,5 @@
   <limit upper="1.570796" lower="-1.570796" effort="100" velocity="100"/>
 </joint>
-<joint name="point" type="revolute">
+<joint name="point" type="fixed">
   <origin xyz="0.035031 -0.020948 8.8e-05" rpy="0 0 0"/>
   <parent link="link6_1"/>

Commit message: l_r_axis_edit

File: urdf/Meta_arm_L.xacro (robot description, xacro)
@@ -6,7 +6,7 @@
 <link name="base_link">
   <inertial>
-    <origin xyz="-0.33486828816047004 -0.05347248420663954 0.3075645449418601" rpy="0 0 0"/>
+    <origin xyz="-0.33328875063083674 0.30962217416987814 0.05141682472682719" rpy="0 0 0"/>
     <mass value="0.07507921631617756"/>
-    <inertia ixx="3.4e-05" iyy="5.2e-05" izz="5.7e-05" ixy="-0.0" iyz="-0.0" ixz="-0.0"/>
+    <inertia ixx="3.4e-05" iyy="5.7e-05" izz="5.2e-05" ixy="0.0" iyz="0.0" ixz="-0.0"/>
   </inertial>
   <visual>
@@ -26,10 +26,10 @@
 <link name="link1_1">
   <inertial>
-    <origin xyz="0.00046123429719080455 0.026932775451258086 -0.020607775962813657" rpy="0 0 0"/>
+    <origin xyz="0.0005001717814695494 -0.020610328537644496 -0.026930416340882047" rpy="0 0 0"/>
     <mass value="0.09072802323891821"/>
-    <inertia ixx="5.6e-05" iyy="5.8e-05" izz="4e-05" ixy="-0.0" iyz="1e-06" ixz="1e-06"/>
-  </inertial>
-  <visual>
-    <origin xyz="0.335107 0.026379 -0.31816" rpy="0 0 0"/>
+    <inertia ixx="5.6e-05" iyy="4e-05" izz="5.8e-05" ixy="1e-06" iyz="-1e-06" ixz="0.0"/>
+  </inertial>
+  <visual>
+    <origin xyz="0.333295 -0.320219 -0.024323" rpy="0 0 0"/>
     <geometry>
       <mesh filename="package://Meta_arm_L_description/meshes/link1_1.stl" scale="0.001 0.001 0.001"/>
@@ -38,5 +38,5 @@
   </visual>
   <collision>
-    <origin xyz="0.335107 0.026379 -0.31816" rpy="0 0 0"/>
+    <origin xyz="0.333295 -0.320219 -0.024323" rpy="0 0 0"/>
     <geometry>
       <mesh filename="package://Meta_arm_L_description/meshes/link1_1.stl" scale="0.001 0.001 0.001"/>
@@ -46,10 +46,10 @@
 <link name="link2_1">
   <inertial>
-    <origin xyz="-0.01872831671678138 -0.001561689883616333 -0.07387427975675265" rpy="0 0 0"/>
+    <origin xyz="-0.019192184742943874 -0.07375769719929967 0.0014429596962129757" rpy="0 0 0"/>
     <mass value="0.1471165597971976"/>
-    <inertia ixx="0.000149" iyy="0.000156" izz="0.000101" ixy="-0.0" iyz="-2e-06" ixz="0.0"/>
-  </inertial>
-  <visual>
-    <origin xyz="0.314977 -0.001075 -0.269687" rpy="0 0 0"/>
+    <inertia ixx="0.000149" iyy="0.000101" izz="0.000156" ixy="0.0" iyz="2e-06" ixz="-0.0"/>
+  </inertial>
+  <visual>
+    <origin xyz="0.313296 -0.271623 0.003008" rpy="0 0 0"/>
     <geometry>
       <mesh filename="package://Meta_arm_L_description/meshes/link2_1.stl" scale="0.001 0.001 0.001"/>
@@ -58,5 +58,5 @@
   </visual>
   <collision>
-    <origin xyz="0.314977 -0.001075 -0.269687" rpy="0 0 0"/>
+    <origin xyz="0.313296 -0.271623 0.003008" rpy="0 0 0"/>
     <geometry>
       <mesh filename="package://Meta_arm_L_description/meshes/link2_1.stl" scale="0.001 0.001 0.001"/>
@@ -66,10 +66,10 @@
 <link name="link3_1">
   <inertial>
-    <origin xyz="-0.0007806403102720849 5.97672584689747e-05 -0.1049169130174851" rpy="0 0 0"/>
-    <mass value="0.10706627889201803"/>
-    <inertia ixx="0.000397" iyy="0.000397" izz="6.8e-05" ixy="-0.0" iyz="1e-06" ixz="-4e-06"/>
-  </inertial>
-  <visual>
-    <origin xyz="0.333523 -0.000586 -0.163572" rpy="0 0 0"/>
+    <origin xyz="-0.001427254193987093 -0.10491003326834535 -6.838068041848614e-05" rpy="0 0 0"/>
+    <mass value="0.10706627889201703"/>
+    <inertia ixx="0.000397" iyy="6.8e-05" izz="0.000397" ixy="-6e-06" iyz="-1e-06" ixz="0.0"/>
+  </inertial>
+  <visual>
+    <origin xyz="0.332498 -0.165624 0.002638" rpy="0 0 0"/>
     <geometry>
       <mesh filename="package://Meta_arm_L_description/meshes/link3_1.stl" scale="0.001 0.001 0.001"/>
@@ -78,5 +78,5 @@
   </visual>
   <collision>
-    <origin xyz="0.333523 -0.000586 -0.163572" rpy="0 0 0"/>
+    <origin xyz="0.332498 -0.165624 0.002638" rpy="0 0 0"/>
     <geometry>
       <mesh filename="package://Meta_arm_L_description/meshes/link3_1.stl" scale="0.001 0.001 0.001"/>
@@ -86,10 +86,10 @@
 <link name="link4_1">
   <inertial>
-    <origin xyz="0.07829896316397977 -0.021020561509984086 -0.00264815215497231" rpy="0 0 0"/>
+    <origin xyz="0.07814907320248449 -0.003130881138898635 0.021503328846025793" rpy="0 0 0"/>
     <mass value="0.13281320983548392"/>
-    <inertia ixx="8.9e-05" iyy="0.000114" izz="0.000116" ixy="-0.0" iyz="-0.0" ixz="-6e-06"/>
-  </inertial>
-  <visual>
-    <origin xyz="0.332521 -0.020998 0.002124" rpy="0 0 0"/>
+    <inertia ixx="8.9e-05" iyy="0.000117" izz="0.000114" ixy="-6e-06" iyz="-0.0" ixz="-0.0"/>
+  </inertial>
+  <visual>
+    <origin xyz="0.332391 7.5e-05 0.02305" rpy="0 0 0"/>
     <geometry>
       <mesh filename="package://Meta_arm_L_description/meshes/link4_1.stl" scale="0.001 0.001 0.001"/>
@@ -98,5 +98,5 @@
   </visual>
   <collision>
-    <origin xyz="0.332521 -0.020998 0.002124" rpy="0 0 0"/>
+    <origin xyz="0.332391 7.5e-05 0.02305" rpy="0 0 0"/>
     <geometry>
       <mesh filename="package://Meta_arm_L_description/meshes/link4_1.stl" scale="0.001 0.001 0.001"/>
@@ -106,7 +106,7 @@
 <link name="link5_1">
   <inertial>
-    <origin xyz="0.11723175095754476 -0.00047610265198036553 0.0007387685571864485" rpy="0 0 0"/>
+    <origin xyz="0.1172289147796068 1.5261168174093082e-05 0.0011987009737727272" rpy="0 0 0"/>
     <mass value="0.09445026816347044"/>
-    <inertia ixx="6e-05" iyy="0.000487" izz="0.000489" ixy="3e-06" iyz="0.0" ixz="-3e-06"/>
+    <inertia ixx="6e-05" iyy="0.000489" izz="0.000487" ixy="-0.0" iyz="-0.0" ixz="-5e-06"/>
   </inertial>
   <visual>
@@ -126,10 +126,10 @@
 <link name="link6_1">
   <inertial>
-    <origin xyz="0.018539706605506658 0.02099956935661064 4.091798251513308e-05" rpy="0 0 0"/>
+    <origin xyz="0.018668706730732707 -7.344937147749836e-05 -0.020885102324875345" rpy="0 0 0"/>
     <mass value="0.029206480233661163"/>
-    <inertia ixx="2.3e-05" iyy="1.1e-05" izz="2.4e-05" ixy="-0.0" iyz="0.0" ixz="-0.0"/>
-  </inertial>
-  <visual>
-    <origin xyz="0.037527 0.021001 0.000158" rpy="0 0 0"/>
+    <inertia ixx="2.3e-05" iyy="2.4e-05" izz="1.1e-05" ixy="0.0" iyz="-0.0" ixz="0.0"/>
+  </inertial>
+  <visual>
+    <origin xyz="0.037656 -7.2e-05 -0.020768" rpy="0 0 0"/>
     <geometry>
       <mesh filename="package://Meta_arm_L_description/meshes/link6_1.stl" scale="0.001 0.001 0.001"/>
@@ -138,5 +138,5 @@
   </visual>
   <collision>
-    <origin xyz="0.037527 0.021001 0.000158" rpy="0 0 0"/>
+    <origin xyz="0.037656 -7.2e-05 -0.020768" rpy="0 0 0"/>
     <geometry>
       <mesh filename="package://Meta_arm_L_description/meshes/link6_1.stl" scale="0.001 0.001 0.001"/>
@@ -146,7 +146,7 @@
 <link name="point_1">
   <inertial>
-    <origin xyz="0.001286507278132388 -5.990973996915515e-07 8.353280042473929e-06" rpy="0 0 0"/>
+    <origin xyz="0.0012865063613372682 -4.4990132036747216e-07 8.501953292352023e-06" rpy="0 0 0"/>
     <mass value="0.0006569528428977276"/>
-    <inertia ixx="0.0" iyy="0.0" izz="0.0" ixy="0.0" iyz="0.0" ixz="0.0"/>
+    <inertia ixx="0.0" iyy="0.0" izz="0.0" ixy="-0.0" iyz="0.0" ixz="0.0"/>
   </inertial>
   <visual>
@@ -165,33 +165,33 @@
 </link>
 <joint name="joint1" type="revolute">
-  <origin xyz="-0.335107 -0.026379 0.31816" rpy="0 0 0"/>
+  <origin xyz="-0.333295 0.320219 0.024323" rpy="0 0 0"/>
   <parent link="base_link"/>
   <child link="link1_1"/>
-  <axis xyz="-0.006145 0.999975 -0.003529"/>
+  <axis xyz="-0.0 -0.003491 -0.999994"/>
   <limit upper="1.570796" lower="-1.570796" effort="100" velocity="100"/>
 </joint>
 <joint name="joint2" type="revolute">
-  <origin xyz="0.02013 0.027454 -0.048473" rpy="0 0 0"/>
+  <origin xyz="0.019999 -0.048596 -0.027331" rpy="0 0 0"/>
   <parent link="link1_1"/>
   <child link="link2_1"/>
-  <axis xyz="0.999962 0.006166 0.006145"/>
+  <axis xyz="1.0 -2.2e-05 0.0"/>
   <limit upper="1.570796" lower="0.0" effort="100" velocity="100"/>
 </joint>
 <joint name="joint3" type="revolute">
-  <origin xyz="-0.018546 -0.000489 -0.106115" rpy="0 0 0"/>
+  <origin xyz="-0.019202 -0.105999 0.00037" rpy="0 0 0"/>
   <parent link="link2_1"/>
   <child link="link3_1"/>
-  <axis xyz="-0.006166 0.003491 0.999975"/>
+  <axis xyz="2.2e-05 0.999994 -0.003491"/>
   <limit upper="2.617994" lower="-2.617994" effort="100" velocity="100"/>
 </joint>
 <joint name="joint4" type="revolute">
-  <origin xyz="0.001002 0.020412 -0.165696" rpy="0 0 0"/>
+  <origin xyz="0.000107 -0.165699 -0.020412" rpy="0 0 0"/>
   <parent link="link3_1"/>
   <child link="link4_1"/>
-  <axis xyz="2.2e-05 0.999994 -0.003491"/>
-  <limit upper="1.745329" lower="-0.872665" effort="100" velocity="100"/>
+  <axis xyz="0.006166 -0.003491 -0.999975"/>
+  <limit upper="1.570796" lower="-0.610866" effort="100" velocity="100"/>
 </joint>
 <joint name="joint5" type="revolute">
-  <origin xyz="0.105998 -0.020999 0.000727" rpy="0 0 0"/>
+  <origin xyz="0.105868 7.4e-05 0.021653" rpy="0 0 0"/>
   <parent link="link4_1"/>
   <child link="link5_1"/>
@@ -200,15 +200,15 @@
 </joint>
 <joint name="joint6" type="revolute">
-  <origin xyz="0.188996 -0.021 0.001239" rpy="0 0 0"/>
+  <origin xyz="0.188867 7.3e-05 0.022165" rpy="0 0 0"/>
   <parent link="link5_1"/>
   <child link="link6_1"/>
-  <axis xyz="-2.2e-05 -0.999994 0.003491"/>
+  <axis xyz="-0.006166 0.003491 0.999975"/>
   <limit upper="1.570796" lower="-1.570796" effort="100" velocity="100"/>
 </joint>
 <joint name="point" type="fixed">
-  <origin xyz="0.035 0.021 0.000142" rpy="0 0 0"/>
+  <origin xyz="0.035129 -7.3e-05 -0.020784" rpy="0 0 0"/>
   <parent link="link6_1"/>
   <child link="point_1"/>
-  <axis xyz="0.999981 -0.0 0.006166"/>
+  <axis xyz="0.999981 0.0 0.006166"/>
   <limit upper="0.001745" lower="0.0" effort="100" velocity="100"/>
 </joint>

File: urdf/Meta_arm_R.xacro (robot description, xacro)
@@ -6,7 +6,7 @@
 <link name="base_link">
   <inertial>
-    <origin xyz="-0.33088647701943896 0.055366724419827235 0.3091965337201203" rpy="0 0 0"/>
+    <origin xyz="-0.3312641243721142 0.30870397524857063 -0.05585487339132518" rpy="0 0 0"/>
     <mass value="0.07507921631617756"/>
-    <inertia ixx="3.4e-05" iyy="5.2e-05" izz="5.7e-05" ixy="-0.0" iyz="0.0" ixz="-0.0"/>
+    <inertia ixx="3.4e-05" iyy="5.7e-05" izz="5.2e-05" ixy="-0.0" iyz="-0.0" ixz="-0.0"/>
   </inertial>
   <visual>
@@ -26,10 +26,10 @@
 <link name="link1_1">
   <inertial>
-    <origin xyz="0.0003216640877543586 -0.02708725297084469 -0.020402070097994662" rpy="0 0 0"/>
-    <mass value="0.09072799201107641"/>
-    <inertia ixx="5.6e-05" iyy="5.8e-05" izz="4e-05" ixy="0.0" iyz="-1e-06" ixz="1e-06"/>
-  </inertial>
-  <visual>
-    <origin xyz="0.33084 -0.028355 -0.320001" rpy="0 0 0"/>
+    <origin xyz="0.00031247585312027537 -0.020402188945389366 0.027087588289717034" rpy="0 0 0"/>
+    <mass value="0.09072799201107642"/>
+    <inertia ixx="5.6e-05" iyy="4e-05" izz="5.8e-05" ixy="1e-06" iyz="1e-06" ixz="-0.0"/>
+  </inertial>
+  <visual>
+    <origin xyz="0.331274 -0.319509 0.028843" rpy="0 0 0"/>
     <geometry>
       <mesh filename="package://Meta_arm_R_description/meshes/link1_1.stl" scale="0.001 0.001 0.001"/>
@@ -38,5 +38,5 @@
   </visual>
   <collision>
-    <origin xyz="0.33084 -0.028355 -0.320001" rpy="0 0 0"/>
+    <origin xyz="0.331274 -0.319509 0.028843" rpy="0 0 0"/>
     <geometry>
       <mesh filename="package://Meta_arm_R_description/meshes/link1_1.stl" scale="0.001 0.001 0.001"/>
@@ -46,10 +46,10 @@
 <link name="link2_1">
   <inertial>
-    <origin xyz="-0.01921036740680765 0.0008469376148304755 -0.07376643698029026" rpy="0 0 0"/>
+    <origin xyz="-0.019099777679982055 -0.07379468679874154 -0.0008758525302789168" rpy="0 0 0"/>
     <mass value="0.1471165597971976"/>
-    <inertia ixx="0.000149" iyy="0.000156" izz="0.000101" ixy="0.0" iyz="2e-06" ixz="-0.0"/>
-  </inertial>
-  <visual>
-    <origin xyz="0.3108 -0.000681 -0.271617" rpy="0 0 0"/>
+    <inertia ixx="0.000149" iyy="0.000101" izz="0.000156" ixy="0.0" iyz="-2e-06" ixz="-0.0"/>
+  </inertial>
+  <visual>
+    <origin xyz="0.311202 -0.271154 0.001139" rpy="0 0 0"/>
     <geometry>
       <mesh filename="package://Meta_arm_R_description/meshes/link2_1.stl" scale="0.001 0.001 0.001"/>
@@ -58,5 +58,5 @@
   </visual>
   <collision>
-    <origin xyz="0.3108 -0.000681 -0.271617" rpy="0 0 0"/>
+    <origin xyz="0.311202 -0.271154 0.001139" rpy="0 0 0"/>
     <geometry>
       <mesh filename="package://Meta_arm_R_description/meshes/link2_1.stl" scale="0.001 0.001 0.001"/>
@@ -66,10 +66,10 @@
 <link name="link3_1">
   <inertial>
-    <origin xyz="-0.0013976754984793005 -0.0008527269650452504 -0.10490304510351446" rpy="0 0 0"/>
+    <origin xyz="-0.0012432407059169148 -0.10490521211286019 0.0008507627627961211" rpy="0 0 0"/>
     <mass value="0.107064701992621"/>
-    <inertia ixx="0.000397" iyy="0.000397" izz="6.9e-05" ixy="0.0" iyz="-4e-06" ixz="-6e-06"/>
-  </inertial>
-  <visual>
-    <origin xyz="0.33 -0.000207 -0.165618" rpy="0 0 0"/>
+    <inertia ixx="0.000397" iyy="6.8e-05" izz="0.000397" ixy="-6e-06" iyz="4e-06" ixz="-0.0"/>
+  </inertial>
+  <visual>
+    <origin xyz="0.330245 -0.165127 0.000694" rpy="0 0 0"/>
     <geometry>
       <mesh filename="package://Meta_arm_R_description/meshes/link3_1.stl" scale="0.001 0.001 0.001"/>
@@ -78,5 +78,5 @@
   </visual>
   <collision>
-    <origin xyz="0.33 -0.000207 -0.165618" rpy="0 0 0"/>
+    <origin xyz="0.330245 -0.165127 0.000694" rpy="0 0 0"/>
     <geometry>
       <mesh filename="package://Meta_arm_R_description/meshes/link3_1.stl" scale="0.001 0.001 0.001"/>
@@ -86,10 +86,10 @@
 <link name="link4_1">
   <inertial>
-    <origin xyz="0.07824995394459477 0.021092636153688817 -0.0032928445732144404" rpy="0 0 0"/>
+    <origin xyz="0.07828568739927477 -0.0031763836143609324 -0.020977037579631326" rpy="0 0 0"/>
     <mass value="0.13281320983548392"/>
-    <inertia ixx="8.9e-05" iyy="0.000114" izz="0.000117" ixy="-0.0" iyz="-0.0" ixz="-6e-06"/>
-  </inertial>
-  <visual>
-    <origin xyz="0.329969 0.021489 -9e-05" rpy="0 0 0"/>
+    <inertia ixx="8.9e-05" iyy="0.000117" izz="0.000114" ixy="-6e-06" iyz="0.0" ixz="0.0"/>
+  </inertial>
+  <visual>
+    <origin xyz="0.33 0.000401 -0.021002" rpy="0 0 0"/>
     <geometry>
       <mesh filename="package://Meta_arm_R_description/meshes/link4_1.stl" scale="0.001 0.001 0.001"/>
@@ -98,5 +98,5 @@
   </visual>
   <collision>
-    <origin xyz="0.329969 0.021489 -9e-05" rpy="0 0 0"/>
+    <origin xyz="0.33 0.000401 -0.021002" rpy="0 0 0"/>
     <geometry>
       <mesh filename="package://Meta_arm_R_description/meshes/link4_1.stl" scale="0.001 0.001 0.001"/>
@@ -106,7 +106,7 @@
 <link name="link5_1">
   <inertial>
-    <origin xyz="0.11723347566727721 0.0006494458120512237 -1.6383683315349354e-05" rpy="0 0 0"/>
-    <mass value="0.09445026816347053"/>
-    <inertia ixx="6e-05" iyy="0.000487" izz="0.000489" ixy="-3e-06" iyz="0.0" ixz="0.0"/>
+    <origin xyz="0.1172342013372355 0.00015775532387740085 -0.00047597503738047383" rpy="0 0 0"/>
+    <mass value="0.09445026816347044"/>
+    <inertia ixx="6e-05" iyy="0.000489" izz="0.000487" ixy="-1e-06" iyz="-0.0" ixz="3e-06"/>
   </inertial>
   <visual>
@@ -126,10 +126,10 @@
 <link name="link6_1">
   <inertial>
-    <origin xyz="0.018570657116001595 -0.0209724087992859 8.810192622033183e-05" rpy="0 0 0"/>
+    <origin xyz="0.01853965708835748 0.0001156099432296103 0.0210001222206634" rpy="0 0 0"/>
     <mass value="0.029206480233661163"/>
-    <inertia ixx="2.3e-05" iyy="1.1e-05" izz="2.4e-05" ixy="0.0" iyz="0.0" ixz="-0.0"/>
-  </inertial>
-  <visual>
-    <origin xyz="0.035031 -0.020948 8.8e-05" rpy="0 0 0"/>
+    <inertia ixx="2.3e-05" iyy="2.4e-05" izz="1.1e-05" ixy="-0.0" iyz="-0.0" ixz="-0.0"/>
+  </inertial>
+  <visual>
+    <origin xyz="0.035 0.00014 0.021" rpy="0 0 0"/>
     <geometry>
       <mesh filename="package://Meta_arm_R_description/meshes/link6_1.stl" scale="0.001 0.001 0.001"/>
@@ -138,5 +138,5 @@
   </visual>
   <collision>
-    <origin xyz="0.035031 -0.020948 8.8e-05" rpy="0 0 0"/>
+    <origin xyz="0.035 0.00014 0.021" rpy="0 0 0"/>
     <geometry>
       <mesh filename="package://Meta_arm_R_description/meshes/link6_1.stl" scale="0.001 0.001 0.001"/>
@@ -146,10 +146,10 @@
 <link name="point_1">
   <inertial>
-    <origin xyz="0.0012867754694881573 2.0555496410046282e-06 -8.654606734118107e-09" rpy="0 0 0"/>
+    <origin xyz="0.0012867756901669193 1.9059888775004724e-06 -1.569636595033508e-07" rpy="0 0 0"/>
     <mass value="0.0006569528428977276"/>
-    <inertia ixx="0.0" iyy="0.0" izz="0.0" ixy="0.0" iyz="-0.0" ixz="-0.0"/>
-  </inertial>
-  <visual>
-    <origin xyz="-0.0 -0.0 -0.0" rpy="0 0 0"/>
+    <inertia ixx="0.0" iyy="0.0" izz="0.0" ixy="0.0" iyz="0.0" ixz="0.0"/>
+  </inertial>
+  <visual>
+    <origin xyz="-0.0 -0.0 0.0" rpy="0 0 0"/>
     <geometry>
       <mesh filename="package://Meta_arm_R_description/meshes/point_1.stl" scale="0.001 0.001 0.001"/>
@@ -158,5 +158,5 @@
   </visual>
   <collision>
-    <origin xyz="-0.0 -0.0 -0.0" rpy="0 0 0"/>
+    <origin xyz="-0.0 -0.0 0.0" rpy="0 0 0"/>
     <geometry>
       <mesh filename="package://Meta_arm_R_description/meshes/point_1.stl" scale="0.001 0.001 0.001"/>
@@ -165,12 +165,12 @@
 </link>
 <joint name="joint1" type="revolute">
-  <origin xyz="-0.33084 0.028355 0.320001" rpy="0 0 0"/>
+  <origin xyz="-0.331274 0.319509 -0.028843" rpy="0 0 0"/>
   <parent link="base_link"/>
   <child link="link1_1"/>
-  <axis xyz="0.001482 -0.99999 0.004202"/>
+  <axis xyz="0.0 0.004202 0.999991"/>
   <limit upper="1.570796" lower="-1.570796" effort="100" velocity="100"/>
 </joint>
 <joint name="joint2" type="revolute">
-  <origin xyz="0.02004 -0.027674 -0.048384" rpy="0 0 0"/>
+  <origin xyz="0.020072 -0.048355 0.027704" rpy="0 0 0"/>
   <parent link="link1_1"/>
   <child link="link2_1"/>
@@ -179,19 +179,19 @@
 </joint>
 <joint name="joint3" type="revolute">
-  <origin xyz="-0.0192 -0.000474 -0.105999" rpy="0 0 0"/>
+  <origin xyz="-0.019043 -0.106027 0.000445" rpy="0 0 0"/>
   <parent link="link2_1"/>
   <child link="link3_1"/>
-  <axis xyz="0.0 0.004202 0.999991"/>
+  <axis xyz="-0.001482 0.99999 -0.004202"/>
   <limit upper="2.617994" lower="-2.617994" effort="100" velocity="100"/>
 </joint>
 <joint name="joint4" type="revolute">
-  <origin xyz="3.1e-05 -0.021696 -0.165528" rpy="0 0 0"/>
+  <origin xyz="0.000245 -0.165528 0.021696" rpy="0 0 0"/>
   <parent link="link3_1"/>
   <child link="link4_1"/>
-  <axis xyz="0.001482 -0.99999 0.004202"/>
-  <limit upper="0.872665" lower="-1.745329" effort="100" velocity="100"/>
+  <axis xyz="0.0 0.004202 0.999991"/>
+  <limit upper="0.610866" lower="-1.570796" effort="100" velocity="100"/>
 </joint>
 <joint name="joint5" type="revolute">
-  <origin xyz="0.105969 0.021157 -8.9e-05" rpy="0 0 0"/>
+  <origin xyz="0.106 6.9e-05 -0.021001" rpy="0 0 0"/>
   <parent link="link4_1"/>
   <child link="link5_1"/>
@@ -200,12 +200,12 @@
 </joint>
 <joint name="joint6" type="revolute">
-  <origin xyz="0.188969 0.02128 -8.9e-05" rpy="0 0 0"/>
+  <origin xyz="0.189 0.000192 -0.021001" rpy="0 0 0"/>
   <parent link="link5_1"/>
   <child link="link6_1"/>
-  <axis xyz="-0.001482 0.99999 -0.004202"/>
+  <axis xyz="-0.0 -0.004202 -0.999991"/>
   <limit upper="1.570796" lower="-1.570796" effort="100" velocity="100"/>
 </joint>
 <joint name="point" type="fixed">
-  <origin xyz="0.035031 -0.020948 8.8e-05" rpy="0 0 0"/>
+  <origin xyz="0.035 0.00014 0.021" rpy="0 0 0"/>
   <parent link="link6_1"/>
   <child link="point_1"/>
