Commit message: gg

File: urdf/Meta_arm_L.xacro (robot description, xacro)
@@ -168,5 +168,5 @@
   <parent link="base_link"/>
   <child link="link1_1"/>
-  <axis xyz="0.999998 -0.001756 3e-06"/>
+  <axis xyz="1.0 0.0 0.0"/>
   <limit upper="1.570796" lower="-1.570796" effort="100" velocity="100"/>
 </joint>
@@ -175,5 +175,5 @@
   <parent link="link1_1"/>
   <child link="link2_1"/>
-  <axis xyz="-0.0 0.001735 0.999998"/>
+  <axis xyz="0.0 0.0 1.0"/>
   <limit upper="1.570796" lower="0.0" effort="100" velocity="100"/>
 </joint>
@@ -182,5 +182,5 @@
   <parent link="link2_1"/>
   <child link="link3_1"/>
-  <axis xyz="0.001756 0.999997 -0.001735"/>
+  <axis xyz="0.0 -1.0 -0.0"/>
   <limit upper="2.617994" lower="-2.617994" effort="100" velocity="100"/>
 </joint>
@@ -189,5 +189,5 @@
   <parent link="link3_1"/>
   <child link="link4_1"/>
-  <axis xyz="0.999979 -0.001745 0.006169"/>
+  <axis xyz="1.0 0.0 0.0"/>
   <limit upper="1.570796" lower="-0.610866" effort="100" velocity="100"/>
 </joint>
@@ -196,5 +196,5 @@
   <parent link="link4_1"/>
   <child link="link5_1"/>
-  <axis xyz="0.006166 -0.001745 -0.999979"/>
+  <axis xyz="0.0 0.0 1.0"/>
   <limit upper="2.617994" lower="-2.617994" effort="100" velocity="100"/>
 </joint>
@@ -203,12 +203,12 @@
   <parent link="link5_1"/>
   <child link="link6_1"/>
-  <axis xyz="-0.999979 0.001745 -0.006169"/>
+  <axis xyz="-1.0 0.0 0.0"/>
   <limit upper="1.570796" lower="-1.570796" effort="100" velocity="100"/>
 </joint>
-<joint name="point" type="fixed">
+<joint name="point" type="revolute">
   <origin xyz="0.020784 2.5e-05 0.035128" rpy="0 0 0"/>
   <parent link="link6_1"/>
   <child link="point_1"/>
-  <axis xyz="-0.006166 0.001745 0.999979"/>
+  <axis xyz="0.0 0.0 0.0"/>
   <limit upper="0.000045" lower="0.0" effort="100" velocity="100"/>
 </joint>

File: urdf/Meta_arm_R.xacro (robot description, xacro)
@@ -168,5 +168,5 @@
   <parent link="base_link"/>
   <child link="link1_1"/>
-  <axis xyz="-0.999999 -0.001482 6e-06"/>
+  <axis xyz="-1.0 0.0 0.0"/>
   <limit upper="1.570796" lower="-1.570796" effort="100" velocity="100"/>
 </joint>
@@ -175,5 +175,5 @@
   <parent link="link1_1"/>
   <child link="link2_1"/>
-  <axis xyz="0.0 0.004202 0.999991"/>
+  <axis xyz="0.0 0.0 1.0"/>
   <limit upper="0.0" lower="-1.570796" effort="100" velocity="100"/>
 </joint>
@@ -182,5 +182,5 @@
   <parent link="link2_1"/>
   <child link="link3_1"/>
-  <axis xyz="-0.001482 0.99999 -0.004202"/>
+  <axis xyz="0.0 -1.0 0.0"/>
   <limit upper="2.617994" lower="-2.617994" effort="100" velocity="100"/>
 </joint>
@@ -189,5 +189,5 @@
   <parent link="link3_1"/>
   <child link="link4_1"/>
-  <axis xyz="-0.999999 -0.001482 6e-06"/>
+  <axis xyz="-1.0 0.0 0.0"/>
   <limit upper="0.610866" lower="-1.570796" effort="100" velocity="100"/>
 </joint>
@@ -196,5 +196,5 @@
   <parent link="link4_1"/>
   <child link="link5_1"/>
-  <axis xyz="-0.0 -0.004202 -0.999991"/>
+  <axis xyz="0.0 0.0 1.0"/>
   <limit upper="2.617994" lower="-2.617994" effort="100" velocity="100"/>
 </joint>
@@ -203,12 +203,12 @@
   <parent link="link5_1"/>
   <child link="link6_1"/>
-  <axis xyz="0.999999 0.001482 -6e-06"/>
+  <axis xyz="1.0 0.0 0.0"/>
   <limit upper="1.570796" lower="-1.570796" effort="100" velocity="100"/>
 </joint>
-<joint name="point" type="fixed">
+<joint name="point" type="revolute">
   <origin xyz="-0.021 0.000116 0.035" rpy="0 0 0"/>
   <parent link="link6_1"/>
   <child link="point_1"/>
-  <axis xyz="0.0 0.004202 0.999991"/>
+  <axis xyz="0.0 0.0 1.0"/>
   <limit upper="0.000045" lower="0.0" effort="100" velocity="100"/>
 </joint>

Commit message: add temp limitation code

File: urdf/Meta_arm_L.xacro (robot description, xacro)
@@ -169,5 +169,5 @@
   <child link="link1_1"/>
   <axis xyz="1.0 0.0 0.0"/>
-  <limit upper="1.570796" lower="-1.570796" effort="100" velocity="100"/>
+  <limit upper="3.141592" lower="0.0" effort="100" velocity="100"/>
 </joint>
 <joint name="joint2" type="revolute">
@@ -176,5 +176,5 @@
   <child link="link2_1"/>
   <axis xyz="0.0 0.0 1.0"/>
-  <limit upper="1.570796" lower="0.0" effort="100" velocity="100"/>
+  <limit upper="1.570796" lower="-1.570796" effort="100" velocity="100"/>
 </joint>
 <joint name="joint3" type="revolute">

File: urdf/Meta_arm_R.xacro (robot description, xacro)
@@ -169,5 +169,5 @@
   <child link="link1_1"/>
   <axis xyz="-1.0 0.0 0.0"/>
-  <limit upper="1.570796" lower="-1.570796" effort="100" velocity="100"/>
+  <limit upper="3.141592" lower="0.0" effort="100" velocity="100"/>
 </joint>
 <joint name="joint2" type="revolute">
@@ -176,5 +176,5 @@
   <child link="link2_1"/>
   <axis xyz="0.0 0.0 1.0"/>
-  <limit upper="0.0" lower="-1.570796" effort="100" velocity="100"/>
+  <limit upper="1.570796" lower="-1.570796" effort="100" velocity="100"/>
 </joint>
 <joint name="joint3" type="revolute">

Commit message: 06/15 final_pr_ver

File: urdf/Meta_arm_L.xacro (robot description, xacro)
@@ -169,5 +169,5 @@
   <child link="link1_1"/>
   <axis xyz="1.0 0.0 0.0"/>
-  <limit upper="3.141592" lower="0.0" effort="100" velocity="100"/>
+  <limit upper="3.141592" lower="-3.141592" effort="100" velocity="100"/>
 </joint>
 <joint name="joint2" type="revolute">

File: urdf/Meta_arm_R.xacro (robot description, xacro)
@@ -169,5 +169,5 @@
   <child link="link1_1"/>
   <axis xyz="-1.0 0.0 0.0"/>
-  <limit upper="3.141592" lower="0.0" effort="100" velocity="100"/>
+  <limit upper="3.141592" lower="-3.141592" effort="100" velocity="100"/>
 </joint>
 <joint name="joint2" type="revolute">
